Commit message: la

File: ros2-workspace/src/robot2_description/src/description/robot2.urdf.xacro (robot description, xacro)
@@ -202,5 +202,5 @@
     <!-- Wheels -->
   <xacro:macro name="wheel" params="prefix x_reflect y_reflect">
-    <link name="${prefix}_link">
+    <link name="${prefix}_wheel">
       <collision>
         <origin xyz="0 0 0" rpy="${pi/2} 0 0"/>
@@ -218,13 +218,13 @@
     <xacro:cylinder_inertia m="1" r="${wheel_radius}" h="${wheel_width}"/>
     </link>
-    <joint name="${prefix}" type="continuous">
+    <joint name="${prefix}_wheel" type="continuous">
       <parent link="base_link"/>
-      <child link="${prefix}_link"/>
+      <child link="${prefix}_wheel"/>
       <origin xyz="${x_reflect*wheel_xoff} ${y_reflect*(base_width/2+wheel_ygap)} ${-wheel_zoff}" rpy="0 0 0"/>
       <axis xyz="0 1 0"/>
     </joint>
   </xacro:macro>
-  <xacro:wheel prefix="left_wheel" x_reflect="-1" y_reflect="1" />
-  <xacro:wheel prefix="right_wheel" x_reflect="-1" y_reflect="-1" />
+  <xacro:wheel prefix="left" x_reflect="-1" y_reflect="1" />
+  <xacro:wheel prefix="right" x_reflect="-1" y_reflect="-1" />
 <!--Gazebo Differential Drive Plugin-->
 <gazebo>
