Commit message: drives

File: ros-workspace/src/robot_launch/urdf/test.urdf.xacro (robot description, xacro)
@@ -172,9 +172,11 @@
      		<origin xyz="0 0 0.54" rpy="1.5708 3.14159 1.5708" />
   </xacro:kinect2>-->
+  <!--
     <xacro:include filename="$(find kinect_v2)/urdf/kinect_v2.urdf.xacro" />
     <xacro:kinect_v2  parent="sensorbar_link">
         <origin xyz="0 0 0.8"
                 rpy="0 0 0" />
-    </xacro:kinect_v2>
+	  </xacro:kinect_v2>
+  -->
  <!--
   <xacro:include filename="$(find robot_launch)/urdf/sensors/kinect2.urdf.xacro" />
@@ -216,5 +218,5 @@
     <xacro:cylinder_inertia m="1" r="${wheel_radius}" h="${wheel_width}"/>
     </link>
-    <joint name="${prefix}_joint" type="continuous">
+    <joint name="${prefix}" type="continuous">
       <parent link="base_link"/>
       <child link="${prefix}_link"/>

File: scripts/test.urdf.xacro (robot description, xacro)
@@ -48,10 +48,12 @@
         <xacro:imu_sensor parent="base_link" xyz="0 0 0.30" rpy="0 0 0">
         </xacro:imu_sensor>
+<!-- The following kinect2_xacro defines the _kinect2_rgb_optical_frame
+        And includes the fixed joint  -->
+	<!-- FIXME
   <xacro:include filename="$(find robot_launch)/urdf/kinect2.urdf.xacro" />
-        <!-- The following kinect2_xacro defines the _kinect2_rgb_optical_frame
-        And includes the fixed joint  -->
-        <xacro:kinect2 parent="base_link" prefix="kinect">
+                <xacro:kinect2 parent="base_link" prefix="kinect">
       		<origin xyz="0 0 0.54" rpy="1.5708 3.14159 1.5708" />
         </xacro:kinect2>
+		-->
   <!-- Robot Footprint -->
   <link name="base_footprint"/>
@@ -81,6 +83,9 @@
     </joint>
   </xacro:macro>
-  <xacro:wheel prefix="drivewhl_l" x_reflect="-1" y_reflect="1" />
+  <!-- <xacro:wheel prefix="drivewhl_l" x_reflect="-1" y_reflect="1" />
   <xacro:wheel prefix="drivewhl_r" x_reflect="-1" y_reflect="-1" />
+  -->
+  <xacro:wheel prefix="left_wheel" x_reflect="-1" y_reflect="1" />
+  <xacro:wheel prefix="right_wheel" x_reflect="-1" y_reflect="-1" />
     <!-- Caster Wheel -->
     <!--
