Commit message: bunch of stuff

File: ros-workspace/src/robot_launch/urdf/imu.urdf.xacro (robot description, xacro)
@@ -36,5 +36,5 @@
             <topic>__default_topic__</topic>
             <plugin name='imu_plugin' filename='libgazebo_ros_imu_sensor.so'>
-                <topicName>/imu/data</topicName>
+                <topicName>imu/data</topicName>
                 <bodyName>imu_sensor_link</bodyName>
                 <frameName>imu_sensor_link</frameName>

File: ros-workspace/src/robot_launch/urdf/kinect2.urdf.xacro (robot description, xacro)
@@ -4,5 +4,5 @@
 <!-- License: GPLv3+ -->
 <robot xmlns:xacro="http://www.ros.org/wiki/xacro" name="kinect2">
-  <xacro:macro name="kinect2" params="prefix parent *origin">
+  <xacro:macro name="kinect2" params="prefix parent">
     <material name="Kinect2Grey">
       <color rgba="0.15 0.15 0.15 1.0"/>
@@ -10,5 +10,6 @@
     <!-- Joint connecting the parent to our frame_in -->
     <joint name="${prefix}_kinect2_in_joint" type="fixed">
-      <xacro:insert_block name="origin"/>
+      <!--<origin xyz="0 0 0.54" rpy="1.5708 3.14159 1.5708" />-->
+      <!-- <xacro:insert_block name="origin"/> -->
       <parent link="${parent}"/>
       <child link="${prefix}_kinect2_rgb_optical_frame"/>
@@ -16,7 +17,10 @@
     <link name="${prefix}_kinect2_rgb_optical_frame">
       <visual>
-        <origin rpy="0 0 0" xyz="0 0 0"/>
+     		<!--<origin xyz="0 0 0" rpy="1.5708 3.14159 1.5708" />-->
+        <!--<origin rpy="0 0 0" xyz="0 0 0"/>-->
         <geometry>
-          <!-- these meshes were exported in mm, so scale back to m -->
+          <!-- these meshes were exported in mm, so scale back to m
+          the mesh has to be turned (camera works fine):      		<origin xyz="0 0 0.54" rpy="1.5708 3.14159 1.5708" />
+          -->
           <mesh filename="package://robot_launch/meshes/kinect2_origin_on_rgb_optical_frame.stl" scale="0.001 0.001 0.001"/>
         </geometry>
@@ -24,5 +28,5 @@
       </visual>
       <collision>
-        <origin xyz="0 0 0" rpy="0 0 0" />
+      		<!--<origin xyz="0 0 0" rpy="1.5708 3.14159 1.5708" />-->
         <geometry>
           <mesh
@@ -31,4 +35,99 @@
       </collision>
     </link>
+    <joint name="${prefix}_kinect2_ir_joint" type="fixed">
+      <parent link="${prefix}_kinect2_rgb_optical_frame"/>
+      <child link="${prefix}_kinect2_ir_optical_frame"/>
+    </joint>
+    <link name="${prefix}_kinect2_ir_optical_frame">
+    </link>
+        <gazebo reference="${prefix}_kinect2_ir_optical_frame">
+            <sensor name="${prefix}_sensor" type="depth">
+                <visualize>true</visualize>
+                <always_on>true</always_on>
+                <update_rate>30.0</update_rate>
+                <camera>
+                    <horizontal_fov>${70.0*3.14/180.0}</horizontal_fov>
+                    <image>
+                        <width>512</width>
+                        <height>424</height>
+                        <format>L8</format>
+                    </image>
+                    <clip>
+                        <near>0.1</near>
+                        <far>8.0</far>
+                    </clip>
+                    <noise>
+                        <!-- Noise is sampled independently per pixel on each frame.
+                        That pixel's noise value is added to each of its color
+                        channels, which at that point lie in the range [0,1]. -->
+                        <type>gaussian</type>
+                        <mean>0.0</mean>
+                        <stddev>0.001</stddev>
+                    </noise>
+                </camera>
+                <plugin name="${prefix}_sensor_controller"                        filename="libgazebo_ros_openni_kinect.so">
+                    <cameraName>/ir/</cameraName>
+                    <alwaysOn>true</alwaysOn>
+                    <updateRate>30.0</updateRate>
+                    <imageTopicName>image_ir_rect</imageTopicName>
+                    <depthImageTopicName>image_depth_rect</depthImageTopicName>
+                    <pointCloudTopicName>points</pointCloudTopicName>
+                    <cameraInfoTopicName>camera_info</cameraInfoTopicName>
+                    <!--<depthImageCameraInfoTopicName>depth/camera_info</depthImageCameraInfoTopicName>-->
+                    <frameName>${prefix}_kinect2_ir_optical_frame</frameName>
+                    <pointCloudCutoff>0.5</pointCloudCutoff>
+                    <pointCloudCutoffMax>4.5</pointCloudCutoffMax>
+                    <baseline>0.1</baseline>
+                    <distortionK1>0.0</distortionK1>
+                    <distortionK2>0.0</distortionK2>
+                    <distortionK3>0.0</distortionK3>
+                    <distortionT1>0.0</distortionT1>
+                    <distortionT2>0.0</distortionT2>
+                    <!--<robotNamespace>${prefix}</robotNamespace>-->
+                </plugin>
+            </sensor>
+        </gazebo>
+        <gazebo reference="${prefix}_kinect2_rgb_optical_frame">
+            <sensor name="${prefix}_camera" type="camera">
+                <visualize>true</visualize>
+                <always_on>true</always_on>
+                <update_rate>30.0</update_rate>
+                <camera name="${prefix}_camera">
+                    <horizontal_fov>${70.0*3.14/180.0}</horizontal_fov>
+                    <image>
+                        <width>512</width>
+                        <height>424</height>
+                        <!--<width>1920</width>
+                        <height>1080</height>-->
+                        <format>R8G8B8</format>
+                    </image>
+                    <clip>
+                        <near>0.02</near>
+                        <far>10.0</far>
+                    </clip>
+                    <noise>
+                        <type>gaussian</type>
+                        <mean>0.0</mean>
+                        <stddev>0.007</stddev>
+                    </noise>
+                </camera>
+                <plugin name="${prefix}_camera_controller"
+                        filename="libgazebo_ros_camera.so">
+                    <alwaysOn>true</alwaysOn>
+                    <update_rate>30.0</update_rate>
+                    <cameraName>/sd/</cameraName>
+                    <imageTopicName>image_color_rect</imageTopicName>
+                    <cameraInfoTopicName>camera_info</cameraInfoTopicName>
+                    <frameName>${prefix}_kinect2_rgb_optical_frame</frameName>
+                    <baseline>0.1</baseline>
+                    <distortionK1>0.0</distortionK1>
+                    <distortionK2>0.0</distortionK2>
+                    <distortionK3>0.0</distortionK3>
+                    <distortionT1>0.0</distortionT1>
+                    <distortionT2>0.0</distortionT2>
+                    <!--<robotNamespace>${prefix}</robotNamespace>-->
+                </plugin>
+            </sensor>
+        </gazebo>
   </xacro:macro>
 </robot>

File: ros-workspace/src/robot_launch/urdf/sensors/kinect2.gazebo.xacro (robot description, xacro)
@@ -28,4 +28,28 @@
         <depthImageCameraInfoTopicName>/${camera_name}/depth/camera_info</depthImageCameraInfoTopicName>
         <pointCloudTopicName>/${camera_name}/depth/points</pointCloudTopicName>
+        <!--
+/kinect2/qhd/camera_info
+/kinect2/qhd/image_color_rect
+/kinect2/qhd/image_depth_rect
+/kinect2/sd/camera_info
+/kinect2/sd/image_color_rect
+/kinect2/sd/image_color_rect/compressed
+/kinect2/sd/image_depth
+/kinect2/sd/image_depth/compressed
+/kinect2/sd/image_depth_rect
+/kinect2/sd/image_depth_rect/compressed
+/kinect2/sd/image_ir
+/kinect2/sd/image_ir/compressed
+/kinect2/sd/image_ir_rect
+/kinect2/sd/image_ir_rect/compressed
+/kinect2/sd/points
+-->
+<!--
+        <imageTopicName>/${camera_name}/sd/image_ir</imageTopicName>
+        <cameraInfoTopicName>/${camera_name}/ir/camera_info</cameraInfoTopicName>
+        <depthImageTopicName>/${camera_name}/sd/image_depth</depthImageTopicName>
+        <depthImageCameraInfoTopicName>/${camera_name}/depth/camera_info</depthImageCameraInfoTopicName>
+        <pointCloudTopicName>/${camera_name}/depth/points</pointCloudTopicName>
+-->
         <frameName>${frame_name}</frameName>
         <pointCloudCutoff>0.5</pointCloudCutoff>

File: ros-workspace/src/robot_launch/urdf/test.urdf.xacro (robot description, xacro)
@@ -12,4 +12,10 @@
       <inertia ixx="${m / 12.0 * (d*d + h*h)}" ixy="0.0" ixz="0.0" iyy="${m / 12.0 * (w*w + h*h)}" iyz="0.0" izz="${m / 12.0 * (w*w + d*d)}"/>
     </inertial>
+  </xacro:macro>
+ <xacro:macro name="sphere_inertia" params="m r">
+    <inertia  ixx="${2*m*r*r/5}" ixy = "0" ixz = "0"
+      iyy="${2*m*r*r/5}" iyz = "0"
+      izz="${2*m*r*r/5}"
+    />
   </xacro:macro>
 <!--kilos lengte breedte hoogte-->
@@ -47,33 +53,11 @@
   <xacro:property name="wheel_xoff" value="0.0"/>
   <xacro:property name="caster_xoff" value="0.14"/>
-<link name="dummy">
-   </link>
-  <joint name="dummy_joint" type="fixed">
-     <parent link="dummy"/>
-     <child link="base_link"/>
-  </joint>
   <!-- Robot Base -->
   <link name="base_link">
   <!-- middle in between wheels -->
-  <!--
-    <visual>
-      <geometry>
-        <box size="0.1 ${base_width} 0.1"/>
-      </geometry>
-     <material name="Gray">  <color rgba="0.5 0.5 0.5 1.0"/>    </material>
-    </visual>
-    -->
-    <xacro:box m="1" w="0.1" h="${base_width}" d="0.1"/>
+   <xacro:box m="40" w="0.1" h="${base_width}" d="0.1"/>
   </link>
   <link name="box_link">
-  <!--
-    <visual>
-      <geometry>
-        <box size="${base_length} ${base_width} ${base_height}"/>
-      </geometry>
-      <material name="Black" />
-    </visual>
-    -->
-    <xacro:box m="5" w="${base_length}" h="${base_width}" d="${base_height}"/>
+      <xacro:box m="5" w="${base_length}" h="${base_width}" d="${base_height}"/>
   </link>
     <joint name="box_joint" type="fixed">
@@ -119,6 +103,6 @@
       <bodyName>gps_link</bodyName>
       <frameId>gps_link</frameId>
-      <topicName>/gps/fix</topicName>
-      <velocityTopicName>/gps/fix_velocity</velocityTopicName>
+      <topicName>gps/fix</topicName>
+      <velocityTopicName>gps/fix_velocity</velocityTopicName>
       <referenceLatitude>-30.06022459407145675</referenceLatitude>
       <referenceLongitude>-51.173913575780311191</referenceLongitude>
@@ -132,4 +116,5 @@
     </plugin>
   </gazebo>
+<!--
 <joint name="laser_joint" type="fixed">
     <origin xyz="0 0.2 0" rpy="0 0 0" />
@@ -167,72 +152,12 @@
           <resolution>0.01</resolution>
         </range>
-<!-- Noise parameters based on published spec for Hokuyo laser
-               achieving "+-30mm" accuracy at range < 10m.  A mean of 0.0m and
-               stddev of 0.01m will put 99.7% of samples within 0.03m of the true
-               reading. -->
-        <!--
-        <noise>
-          <type>gaussian</type>
-                    <mean>0.0</mean>
-          <stddev>0.01</stddev>
-        </noise>
-        -->
       </ray>
       <plugin name="gazebo_ros_head_hokuyo_controller" filename="libgazebo_ros_laser.so">
-        <topicName>/rrbot/laser/scan</topicName>
+        <topicName>laser/scan</topicName>
         <frameName>laser</frameName>
       </plugin>
     </sensor>
 </gazebo>
-<joint name="ir_front_joint" type="fixed">
-    <axis xyz="0 1 0" />
-    <origin rpy="0 0 0" xyz="0.5 0 0" />
-    <parent link="sensorbar_link"/>
-    <child link="base_ir_front"/>
-</joint>
-<link name="base_ir_front">
-    <collision>
-      <origin xyz="0 0 0" rpy="0 0 0"/>
-      <geometry>
-        <box size="0.01 0.01 0.01"/>
-      </geometry>
-    </collision>
-    <visual>
-      <origin xyz="0 0 0" rpy="0 0 0"/>
-      <geometry>
-        <box size="0.01 0.01 0.01"/>
-      </geometry>
-    </visual>
-    <inertial>
-      <mass value="1e-5" />
-      <origin xyz="0 0 0" rpy="0 0 0"/>
-      <inertia ixx="1e-6" ixy="0" ixz="0" iyy="1e-6" iyz="0"      izz="1e-6" />
-    </inertial>
-</link>
-<joint name="sonar_front_joint" type="fixed">
-    <axis xyz="0 1 0" />
-    <origin rpy="0 0 0" xyz="0.5 0 0.25" />
-    <parent link="sensorbar_link"/>
-    <child link="base_sonar_front"/>
-</joint>
-<link name="base_sonar_front">
-    <collision>
-      <origin xyz="0 0 0" rpy="0 0 0"/>
-      <geometry>
-        <box size="0.01 0.01 0.01"/>
-      </geometry>
-    </collision>
-    <visual>
-      <origin xyz="0 0 0" rpy="0 0 0"/>
-      <geometry>
-        <box size="0.01 0.01 0.01"/>
-      </geometry>
-    </visual>
-    <inertial>
-      <mass value="1e-5" />
-      <origin xyz="0 0 0" rpy="0 0 0"/>
-      <inertia ixx="1e-6" ixy="0" ixz="0" iyy="1e-6" iyz="0" izz="1e-6" />
-    </inertial>
- </link>
+-->
   <xacro:include filename="$(find robot_launch)/urdf/imu.urdf.xacro" />
         <!-- The following kinect2_xacro defines the _kinect2_rgb_optical_frame
@@ -242,16 +167,22 @@
 <!--          The following kinect2_xacro defines the _kinect2_rgb_optical_frame
         And includes the fixed joint
-  <xacro:include filename="$(find robot_launch)/urdf/kinect2.urdf.xacro" />
-        <xacro:kinect2 parent="base_link" prefix="kinect">
-      		<origin xyz="0 0 0.54" rpy="1.5708 3.14159 1.5708" />
-        </xacro:kinect2>
--->
+        -->
+  <!--<xacro:include filename="$(find robot_launch)/urdf/kinect2.urdf.xacro" />
+        <xacro:kinect2 parent="sensorbar_link" prefix="kinect2" >
+     		<origin xyz="0 0 0.54" rpy="1.5708 3.14159 1.5708" />
+  </xacro:kinect2>-->
+    <xacro:include filename="$(find kinect_v2)/urdf/kinect_v2.urdf.xacro" />
+    <xacro:kinect_v2  parent="sensorbar_link">
+        <origin xyz="0 0 0.8"
+                rpy="0 0 0" />
+    </xacro:kinect_v2>
+ <!--
   <xacro:include filename="$(find robot_launch)/urdf/sensors/kinect2.urdf.xacro" />
   <xacro:kinect2 parent="sensorbar_link" name="KinectSensor2">
-   <!-- <origin xyz="0 0 0.54" rpy="1.5708 3.14159 1.5708" /> -->
     <origin xyz="0 0 0.54" rpy="0 0 0" />
   </xacro:kinect2>
+ -->
   <!-- Robot Footprint -->
-  <link name="base_footprint">
+  <link name="robot_footprint">
   <inertial>
          <mass value="10"/>
@@ -259,7 +190,10 @@
    </inertial>
   </link>
+  <gazebo reference="robot_footprint">
+    <material>Gazebo/Orange</material>
+  </gazebo>
   <joint name="base_joint" type="fixed">
     <parent link="base_link"/>
-    <child link="base_footprint"/>
+    <child link="robot_footprint"/>
     <origin xyz="0.0 0.0 ${-(wheel_radius+wheel_zoff)}" rpy="0 0 0"/>
   </joint>
@@ -312,5 +246,5 @@
     <visual>
       <geometry>
-        <sphere radius="${(wheel_radius+wheel_zoff-(base_height/2))}"/>
+        <sphere radius="${wheel_radius / 2}"/>
       </geometry>
       <material name="Cyan">
@@ -318,9 +252,15 @@
       </material>
     </visual>
+    <collision>
+      <geometry>
+        <sphere radius="${wheel_radius / 2}"/>
+      </geometry>
+    </collision>
+    <xacro:sphere_inertia m="10.3" r="${wheel_radius / 2}"/>
   </link>
   <joint name="caster_joint" type="fixed">
     <parent link="base_link"/>
     <child link="front_caster"/>
-    <origin xyz="${caster_xoff} 0.0 0.1" rpy="0 0 0"/>
+    <origin xyz="${base_length - base_xoff - 0.2} 0.0 ${0 - (wheel_radius / 2)}" rpy="0 0 0"/>
   </joint>
       <gazebo>
